Commit message: Change robot orientation with viscotec

File: ramsai_description/urdf/iiwa14.urdf.xacro (robot description, xacro)
@@ -271,5 +271,5 @@
     </joint>
     <joint name="${prefix}joint_a7-tip" type="fixed">
-        <origin rpy="0 ${alpha} 0" xyz="${sin(alpha)*(l-0.0264)} 0.0 ${dz+cos(alpha)*(l-0.0264)}"/> <!--0.154-->
+        <origin rpy="0 ${alpha} ${math.pi}" xyz="${sin(alpha)*(l-0.0264)} 0.0 ${dz+cos(alpha)*(l-0.0264)}"/> <!--0.154-->
         <parent link="${prefix}link_7"/>
         <child link="${prefix}tip"/>
@@ -277,5 +277,5 @@
     </joint>
     <joint name="${prefix}extruder" type="fixed">
-        <origin rpy="0 0 -1.57" xyz="0.0 0.0 0.0"/> <!--0.154-->
+        <origin rpy="0 0 0" xyz="0.0 0.0 0.0"/> <!--0.154-->
         <parent link="${prefix}tip"/>
         <child link="${prefix}tool0"/>
